Commit message: removed all warning and cleanup, robot still not moving

File: sandbox/team_members/pudumula/ros/gazebo_ws/src/mybot_description/urdf/macros.xacro (robot description, xacro)
@@ -51,15 +51,17 @@
       <parent link="chassis"/>
       <child link="${lr}_wheel"/>
-    <origin xyz="${-wheelPos+chassisLength/2} ${tY*wheelWidth/2+tY*chassisWidth/2} ${wheelRadius}" rpy="0 0 0" />
+      <origin xyz="${-wheelPos+chassisLength/2} ${tY*wheelWidth/2+tY*chassisWidth/2} ${wheelRadius}" rpy="0 0 0" />
       <axis xyz="0 1 0" rpy="0 0 0" />
-      <limit effort="100" velocity="100"/>
-      <joint_properties damping="0.0" friction="0.0"/>
+      <limit effort="10000" velocity="1000"/>
+      <joint_properties damping="1.0" friction="1.0"/>
     </joint>
     <transmission name="${lr}_trans">
       <type>transmission_interface/SimpleTransmission</type>
-      <joint name="${lr}_wheel_hinge"/>
+      <joint name="${lr}_wheel_hinge">
+        <hardwareInterface>EffortJointInterface</hardwareInterface>
+      </joint>
       <actuator name="${lr}Motor">
         <hardwareInterface>EffortJointInterface</hardwareInterface>
-        <mechanicalReduction>10</mechanicalReduction>
+        <mechanicalReduction>1</mechanicalReduction>
       </actuator>
     </transmission>

File: sandbox/team_members/pudumula/ros/gazebo_ws/src/mybot_description/urdf/mybot.xacro (robot description, xacro)
@@ -17,7 +17,7 @@
  	<xacro:include filename="$(find mybot_description)/urdf/materials.xacro" />
  	<xacro:include filename="$(find mybot_description)/urdf/macros.xacro" />
-  <link name="footprint" />
+  <link name="world" />
   <joint name="base_joint" type="fixed">
-    <parent link="footprint"/>
+    <parent link="world"/>
     <child link="chassis"/>
   </joint>
@@ -39,5 +39,5 @@
     			<origin xyz="0 0 ${wheelRadius}" rpy="0 0 0"/>
     			<mass value="${chassisMass}"/>
-    			<box_inertia m="${chassisMass}" x="${chassisLength}" y="${chassisWidth}" z="${chassisHeight}"/>
+    			<xacro:box_inertia m="${chassisMass}" x="${chassisLength}" y="${chassisWidth}" z="${chassisHeight}"/>
   		</inertial>
 	</link>
@@ -63,8 +63,8 @@
       <origin xyz="${casterRadius-chassisLength/2} 0 ${casterRadius-chassisHeight+wheelRadius}" rpy="0 0 0"/>
       <mass value="${casterMass}"/>
-      <sphere_inertia m="${casterMass}" r="${casterRadius}"/>
+      <xacro:sphere_inertia m="${casterMass}" r="${casterRadius}"/>
     </inertial>
   </link>
-  <wheel lr="left" tY="1"/>
-  <wheel lr="right" tY="-1"/>
+  <xacro:wheel lr="left" tY="1"/>
+  <xacro:wheel lr="right" tY="-1"/>
 </robot>
